Commit message: [cpp] change joint-limits to model class + temporary fix for specificities

File: unitTesting/two_link.urdf (robot description, URDF)
Before this commit: robot test_two_link, 3 links, 2 joints
Links:
- added link CHILD3
Joints:
- added joint FRAMEJOINT1: type fixed, parent CHILD2, child CHILD3, origin xyz=0 0 -0.16 rpy=0 0 0
